File: Flashback2.kicad_sch (KiCad schematic)
At the start: 241 parts, among them J1 0, J1 Barrel_Jack, J10 0, J11 0, J12 0, J13 0, J14 0, J15 0, J16 0, J17 0, J18 0, J19 0, J2 0, J20 0, J21 0, J22 0, J23 0, J24 0, J25 0, J26 0, J3 0, J4 0, J5 0, J6 0, J7 0, J8 0, J9 0, Q1 MMBT3904, Q2 MMBT3904, SW1 BW/COLOR, SW2 LEFT DIFFICULTY, SW3 RIGHT DIFFICULTY, SW4 SELECT, SW5 RESET, SW6 POWER, U1 Michele, U2 Game ROM, U3 L7805, U4 SE5119AKN, X1 14.318MHz

Commit message: Add files via upload
Parts:
- added TP100, TP99: ~, symbol Connector:TestPoint_Small
Connections:
- net GND: now also TP100.1, TP99.1
Changed lines of the file:
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@@
 	)
 	(junction
+		(at 116.84 44.45)
+		(diameter 0)
+		(color 0 0 0 0)
+	)
+	(junction
 		(at 132.08 172.72)
 		(diameter 0)
@@
 	)
 	(junction
-		(at 123.19 44.45)
+		(at 121.92 44.45)
 		(diameter 0)
 		(color 0 0 0 0)
@@
 	)
 	(junction
-		(at 118.11 46.99)
-		(diameter 0)
-		(color 0 0 0 0)
-	)
-	(junction
 		(at 351.79 196.85)
 		(diameter 0)
@@
 	)
 	(junction
-		(at 120.65 44.45)
+		(at 119.38 44.45)
 		(diameter 0)
 		(color 0 0 0 0)
@@
 	)
 	(junction
+		(at 116.84 46.99)
+		(diameter 0)
+		(color 0 0 0 0)
+	)
+	(junction
 		(at 147.32 142.24)
 		(diameter 0)
@@
 	)
 	(junction
-		(at 118.11 44.45)
+		(at 83.82 154.94)
 		(diameter 0)
 		(color 0 0 0 0)
 	)
 	(junction
-		(at 83.82 154.94)
+		(at 359.41 213.36)
 		(diameter 0)
 		(color 0 0 0 0)
 	)
 	(junction
-		(at 359.41 213.36)
+		(at 124.46 44.45)
+		(diameter 0)
+		(color 0 0 0 0)
+	)
+	(junction
+		(at 127 44.45)
 		(diameter 0)
 		(color 0 0 0 0)
@@
 	(wire
 		(pts
-			(xy 115.57 39.37) (xy 118.11 39.37)
+			(xy 115.57 39.37) (xy 116.84 39.37)
 		)
 		(stroke
@@
 		)
 	)
+	(wire
+		(pts
+			(xy 124.46 44.45) (xy 127 44.45)
+		)
+		(stroke
+			(width 0)
+			(type default)
+		)
+	)
 	(bus
 		(pts
@@
 		)
 	)
+	(wire
+		(pts
+			(xy 127 44.45) (xy 129.54 44.45)
+		)
+		(stroke
+			(width 0)
+			(type default)
+		)
+	)
 	(bus
 		(pts
@@
 	(wire
 		(pts
-			(xy 118.11 46.99) (xy 118.11 57.15)
+			(xy 116.84 46.99) (xy 116.84 57.15)
 		)
 		(stroke
@@
 	(wire
 		(pts
+			(xy 116.84 46.99) (xy 128.27 46.99)
+		)
+		(stroke
+			(width 0)
+			(type default)
+		)
+	)
+	(wire
+		(pts
 			(xy 285.75 55.88) (xy 285.75 58.42)
 		)
@@
 	(wire
 		(pts
-			(xy 118.11 44.45) (xy 118.11 46.99)
+			(xy 116.84 44.45) (xy 116.84 46.99)
 		)
 		(stroke
@@
 	(wire
 		(pts
-			(xy 118.11 44.45) (xy 120.65 44.45)
-		)
-		(stroke
-			(width 0)
-			(type default)
-		)
-	)
-	(wire
-		(pts
 			(xy 153.67 135.89) (xy 177.8 135.89)
 		)
@@
 	(wire
 		(pts
-			(xy 118.11 46.99) (xy 128.27 46.99)
-		)
-		(stroke
-			(width 0)
-			(type default)
-		)
-	)
-	(wire
-		(pts
 			(xy 45.72 226.06) (xy 50.8 226.06)
 		)
@@
 		)
 	)
+	(wire
+		(pts
+			(xy 116.84 44.45) (xy 119.38 44.45)
+		)
+		(stroke
+			(width 0)
+			(type default)
+		)
+	)
 	(bus
 		(pts
@@
 	(wire
 		(pts
-			(xy 123.19 44.45) (xy 129.54 44.45)
+			(xy 121.92 44.45) (xy 124.46 44.45)
 		)
 		(stroke
@@
 	(wire
 		(pts
-			(xy 118.11 39.37) (xy 118.11 44.45)
+			(xy 116.84 39.37) (xy 116.84 44.45)
 		)
 		(stroke
@@
 	(wire
 		(pts
-			(xy 120.65 44.45) (xy 123.19 44.45)
+			(xy 119.38 44.45) (xy 121.92 44.45)
 		)
 		(stroke
@@
 	(symbol
 		(lib_id "Connector:TestPoint_Small")
+		(at 124.46 44.45 90)
+		(unit 1)
+		(exclude_from_sim no)
+		(in_bom yes)
+		(on_board yes)
+		(dnp no)
+		(property "Reference" "TP99"
+			(at 121.158 39.37 90)
+			(effects
+				(font
+					(size 1.27 1.27)
+				)
+				(hide yes)
+			)
+		)
+		(property "Value" "~"
+			(at 122.682 43.434 90)
+			(effects
+				(font
+					(size 1.27 1.27)
+				)
+			)
+		)
+		(property "Footprint" ""
+			(at 124.46 39.37 0)
+			(effects
+				(font
+					(size 1.27 1.27)
+				)
+				(hide yes)
+			)
+		)
+		(property "Datasheet" "~"
+			(at 124.46 39.37 0)
+			(effects
+				(font
+					(size 1.27 1.27)
+				)
+				(hide yes)
+			)
+		)
+		(property "Description" ""
+			(at 124.46 44.45 0)
+			(effects
+				(font
+					(size 1.27 1.27)
+				)
+				(hide yes)
+			)
+		)
+		(pin "1"
+		)
+		(instances
+			(project "Flashback2"
+				(path "/93745d60-cfe0-4df5-ab28-b8cbe01a455e"
+					(reference "TP99")
+					(unit 1)
+				)
+			)
+		)
+	)
+	(symbol
+		(lib_id "Connector:TestPoint_Small")
 		(at 153.67 142.24 90)
 		(unit 1)
@@
 	(symbol
 		(lib_id "power:GND")
-		(at 118.11 57.15 0)
+		(at 116.84 57.15 0)
 		(unit 1)
 		(exclude_from_sim no)
@@
 		(dnp no)
 		(property "Reference" "#PWR034"
-			(at 118.11 63.5 0)
+			(at 116.84 63.5 0)
 			(effects
 				(font
@@
 		)
 		(property "Value" "GND"
-			(at 118.11 60.96 0)
+			(at 116.84 60.96 0)
 			(effects
 				(font
@@
 		)
 		(property "Footprint" ""
-			(at 118.11 57.15 0)
+			(at 116.84 57.15 0)
 			(effects
 				(font
@@
 		)
 		(property "Datasheet" ""
-			(at 118.11 57.15 0)
+			(at 116.84 57.15 0)
 			(effects
 				(font
@@
 		)
 		(property "Description" ""
-			(at 118.11 57.15 0)
+			(at 116.84 57.15 0)
 			(effects
 				(font
@@
 	(symbol
 		(lib_id "Connector:TestPoint_Small")
-		(at 120.65 44.45 90)
+		(at 119.38 44.45 90)
 		(unit 1)
 		(exclude_from_sim no)
@@
 		(dnp no)
 		(property "Reference" "TP89"
-			(at 117.348 39.37 90)
+			(at 116.078 39.37 90)
 			(effects
 				(font
@@
 		)
 		(property "Value" "~"
-			(at 118.872 43.434 90)
+			(at 117.602 43.434 90)
 			(effects
 				(font
@@
 		)
 		(property "Footprint" ""
-			(at 120.65 39.37 0)
+			(at 119.38 39.37 0)
 			(effects
 				(font
@@
 		)
 		(property "Datasheet" "~"
-			(at 120.65 39.37 0)
+			(at 119.38 39.37 0)
 			(effects
 				(font
@@
 		)
 		(property "Description" ""
-			(at 120.65 44.45 0)
+			(at 119.38 44.45 0)
 			(effects
 				(font
@@
 	(symbol
 		(lib_id "Connector:TestPoint_Small")
-		(at 123.19 44.45 90)
+		(at 121.92 44.45 90)
 		(unit 1)
 		(exclude_from_sim no)
@@
 		(dnp no)
 		(property "Reference" "TP90"
-			(at 119.888 39.37 90)
+			(at 118.618 39.37 90)
 			(effects
 				(font
@@
 		)
 		(property "Value" "~"
-			(at 121.412 43.434 90)
+			(at 120.142 43.434 90)
 			(effects
 				(font
@@
 		)
 		(property "Footprint" ""
-			(at 123.19 39.37 0)
+			(at 121.92 39.37 0)
 			(effects
 				(font
@@
 		)
 		(property "Datasheet" "~"
-			(at 123.19 39.37 0)
+			(at 121.92 39.37 0)
 			(effects
 				(font
@@
 		)
 		(property "Description" ""
-			(at 123.19 44.45 0)
+			(at 121.92 44.45 0)
 			(effects
 				(font
@@
 					(unit 1)
 				)
+			)
+		)
+	)
+	(symbol
+		(lib_id "Connector:TestPoint_Small")
+		(at 127 44.45 90)
+		(unit 1)
+		(exclude_from_sim no)
+		(in_bom yes)
+		(on_board yes)
+		(dnp no)
+		(property "Reference" "TP100"
+			(at 123.698 39.37 90)
+			(effects
+				(font
+					(size 1.27 1.27)
+				)
+				(hide yes)
+			)
+		)
+		(property "Value" "~"
+			(at 125.222 43.434 90)
+			(effects
+				(font
+					(size 1.27 1.27)
+				)
+			)
+		)
+		(property "Footprint" ""
+			(at 127 39.37 0)
+			(effects
+				(font
+					(size 1.27 1.27)
+				)
+				(hide yes)
+			)
+		)
+		(property "Datasheet" "~"
+			(at 127 39.37 0)
+			(effects
+				(font
+					(size 1.27 1.27)
+				)
+				(hide yes)
+			)
+		)
+		(property "Description" ""
+			(at 127 44.45 0)
+			(effects
+				(font
+					(size 1.27 1.27)
+				)
+				(hide yes)
+			)
+		)
+		(pin "1"
+		)
+		(instances
+			(project "Flashback2"
+				(path "/93745d60-cfe0-4df5-ab28-b8cbe01a455e"
+					(reference "TP100")
+					(unit 1)
+				)
